Commit message: Change pkg name

File: catkin_ws/src/grinding_descriptions/urdf/cobotta.urdf (robot description, URDF)
Before this commit: robot stdcb, 9 links, 8 joints
Links:
- link pestle: geometry visual mesh filename=package://grinding_descriptions/mesh/jig_pestle_170.stl

File: catkin_ws/src/grinding_descriptions/urdf/cobotta.urdf.xacro (robot description, xacro)
@@ -27,4 +27,4 @@
     <xacro:cobotta_macro joint="joint_5" parent="J4" child="J5" joint_type="revolute" origin_xyz="0 -0.02 0.52225" axis="0 1 0" lower="-1.65806278939461" upper="2.35619449019234" file_path="package://denso_descr/stdcb_description/J5.stl"/>
     <xacro:cobotta_macro joint="joint_6" parent="J5" child="J6" joint_type="revolute" origin_xyz="0 -0.0445 0.042" axis="0 0 1" lower="-2.96705972839036" upper="2.96705972839036" file_path="package://denso_descr/stdcb_description/J6.stl"/>
-    <xacro:cobotta_macro joint="joint_pestle" parent="J6" child="pestle" joint_type="fixed" origin_xyz="0 0 0" axis="0 0 0" upper="0" lower="0" file_path="package://kek_scene_description/mesh/jig_pestle_170.stl"/>
+    <xacro:cobotta_macro joint="joint_pestle" parent="J6" child="pestle" joint_type="fixed" origin_xyz="0 0 0" axis="0 0 0" upper="0" lower="0" file_path="package://grinding_descriptions/mesh/jig_pestle_170.stl"/>
 </robot>

File: catkin_ws/src/grinding_descriptions/urdf/inc/ur10_macro.xacro (robot description, xacro)
@@ -3,7 +3,7 @@
   <!--
     Convenience wrapper for the 'ur_robot' macro which provides default values
-    for the various "parameters files" parameters for a UR5.
+    for the various "parameters files" parameters for a UR10.
     This file can be used when composing a more complex scene with one or more
-    UR5 robots.
+    UR10 robots.
     While the generic 'ur_robot' macro could also be used, it would require
     the user to provide values for all parameters, as that macro does not set
@@ -17,11 +17,11 @@
           real robot.
   -->
-  <xacro:macro name="ur5_robot"
+  <xacro:macro name="ur10_robot"
     params="
    prefix
-   joint_limits_parameters_file:='$(find kek_scene_description)/config/ur5/joint_limits.yaml'
-   kinematics_parameters_file:='$(find kek_scene_description)/config/ur5/default_kinematics.yaml'
-   physical_parameters_file:='$(find kek_scene_description)/config/ur5/physical_parameters.yaml'
-   visual_parameters_file:='$(find kek_scene_description)/config/ur5/visual_parameters.yaml'
+   joint_limits_parameters_file:='$(find grinding_descriptions)/config/ur10/joint_limits.yaml'
+   kinematics_parameters_file:='$(find grinding_descriptions)/config/ur10/default_kinematics.yaml'
+   physical_parameters_file:='$(find grinding_descriptions)/config/ur10/physical_parameters.yaml'
+   visual_parameters_file:='$(find grinding_descriptions)/config/ur10/visual_parameters.yaml'
    transmission_hw_interface:=hardware_interface/PositionJointInterface
    safety_limits:=false
@@ -29,5 +29,5 @@
    safety_k_position:=20"
   >
-    <xacro:include filename="$(find kek_scene_description)/urdf/inc/ur_macro.xacro" />
+    <xacro:include filename="$(find grinding_descriptions)/urdf/inc/ur_macro.xacro" />
     <xacro:ur_robot
       prefix="${prefix}"

File: catkin_ws/src/grinding_descriptions/urdf/inc/ur10e_macro.xacro (robot description, xacro)
@@ -3,7 +3,7 @@
   <!--
     Convenience wrapper for the 'ur_robot' macro which provides default values
-    for the various "parameters files" parameters for a UR3.
+    for the various "parameters files" parameters for a UR10e.
     This file can be used when composing a more complex scene with one or more
-    UR3 robots.
+    UR10e robots.
     While the generic 'ur_robot' macro could also be used, it would require
     the user to provide values for all parameters, as that macro does not set
@@ -17,11 +17,11 @@
           real robot.
   -->
-  <xacro:macro name="ur3_robot"
+  <xacro:macro name="ur10e_robot"
     params="
    prefix
-   joint_limits_parameters_file:='$(find kek_scene_description)/config/ur3/joint_limits.yaml'
-   kinematics_parameters_file:='$(find kek_scene_description)/config/ur3/default_kinematics.yaml'
-   physical_parameters_file:='$(find kek_scene_description)/config/ur3/physical_parameters.yaml'
-   visual_parameters_file:='$(find kek_scene_description)/config/ur3/visual_parameters.yaml'
+   joint_limits_parameters_file:='$(find grinding_descriptions)/config/ur10e/joint_limits.yaml'
+   kinematics_parameters_file:='$(find grinding_descriptions)/config/ur10e/default_kinematics.yaml'
+   physical_parameters_file:='$(find grinding_descriptions)/config/ur10e/physical_parameters.yaml'
+   visual_parameters_file:='$(find grinding_descriptions)/config/ur10e/visual_parameters.yaml'
    transmission_hw_interface:=hardware_interface/PositionJointInterface
    safety_limits:=false
@@ -29,5 +29,5 @@
    safety_k_position:=20"
   >
-    <xacro:include filename="$(find kek_scene_description)/urdf/inc/ur_macro.xacro" />
+    <xacro:include filename="$(find grinding_descriptions)/urdf/inc/ur_macro.xacro" />
     <xacro:ur_robot
       prefix="${prefix}"

File: catkin_ws/src/grinding_descriptions/urdf/inc/ur16e_macro.xacro (robot description, xacro)
@@ -20,8 +20,8 @@
     params="
    prefix
-   joint_limits_parameters_file:='$(find kek_scene_description)/config/ur16e/joint_limits.yaml'
-   kinematics_parameters_file:='$(find kek_scene_description)/config/ur16e/default_kinematics.yaml'
-   physical_parameters_file:='$(find kek_scene_description)/config/ur16e/physical_parameters.yaml'
-   visual_parameters_file:='$(find kek_scene_description)/config/ur16e/visual_parameters.yaml'
+   joint_limits_parameters_file:='$(find grinding_descriptions)/config/ur16e/joint_limits.yaml'
+   kinematics_parameters_file:='$(find grinding_descriptions)/config/ur16e/default_kinematics.yaml'
+   physical_parameters_file:='$(find grinding_descriptions)/config/ur16e/physical_parameters.yaml'
+   visual_parameters_file:='$(find grinding_descriptions)/config/ur16e/visual_parameters.yaml'
    transmission_hw_interface:=hardware_interface/PositionJointInterface
    safety_limits:=false
@@ -29,5 +29,5 @@
    safety_k_position:=20"
   >
-    <xacro:include filename="$(find kek_scene_description)/urdf/inc/ur_macro.xacro" />
+    <xacro:include filename="$(find grinding_descriptions)/urdf/inc/ur_macro.xacro" />
     <xacro:ur_robot
       prefix="${prefix}"

File: catkin_ws/src/grinding_descriptions/urdf/inc/ur3_macro.xacro (robot description, xacro)
@@ -3,7 +3,7 @@
   <!--
     Convenience wrapper for the 'ur_robot' macro which provides default values
-    for the various "parameters files" parameters for a UR5e.
+    for the various "parameters files" parameters for a UR3.
     This file can be used when composing a more complex scene with one or more
-    UR5e robots.
+    UR3 robots.
     While the generic 'ur_robot' macro could also be used, it would require
     the user to provide values for all parameters, as that macro does not set
@@ -17,11 +17,11 @@
           real robot.
   -->
-  <xacro:macro name="ur5e_robot"
+  <xacro:macro name="ur3_robot"
     params="
    prefix
-   joint_limits_parameters_file:='$(find kek_scene_description)/config/ur5e/joint_limits.yaml'
-   kinematics_parameters_file:='$(find kek_scene_description)/config/ur5e/default_kinematics.yaml'
-   physical_parameters_file:='$(find kek_scene_description)/config/ur5e/physical_parameters.yaml'
-   visual_parameters_file:='$(find kek_scene_description)/config/ur5e/visual_parameters.yaml'
+   joint_limits_parameters_file:='$(find grinding_descriptions)/config/ur3/joint_limits.yaml'
+   kinematics_parameters_file:='$(find grinding_descriptions)/config/ur3/default_kinematics.yaml'
+   physical_parameters_file:='$(find grinding_descriptions)/config/ur3/physical_parameters.yaml'
+   visual_parameters_file:='$(find grinding_descriptions)/config/ur3/visual_parameters.yaml'
    transmission_hw_interface:=hardware_interface/PositionJointInterface
    safety_limits:=false
@@ -29,5 +29,5 @@
    safety_k_position:=20"
   >
-    <xacro:include filename="$(find kek_scene_description)/urdf/inc/ur_macro.xacro" />
+    <xacro:include filename="$(find grinding_descriptions)/urdf/inc/ur_macro.xacro" />
     <xacro:ur_robot
       prefix="${prefix}"

File: catkin_ws/src/grinding_descriptions/urdf/inc/ur3e_macro.xacro (robot description, xacro)
@@ -20,8 +20,8 @@
     params="
    prefix
-   joint_limits_parameters_file:='$(find kek_scene_description)/config/ur3e/joint_limits.yaml'
-   kinematics_parameters_file:='$(find kek_scene_description)/config/ur3e/default_kinematics.yaml'
-   physical_parameters_file:='$(find kek_scene_description)/config/ur3e/physical_parameters.yaml'
-   visual_parameters_file:='$(find kek_scene_description)/config/ur3e/visual_parameters.yaml'
+   joint_limits_parameters_file:='$(find grinding_descriptions)/config/ur3e/joint_limits.yaml'
+   kinematics_parameters_file:='$(find grinding_descriptions)/config/ur3e/default_kinematics.yaml'
+   physical_parameters_file:='$(find grinding_descriptions)/config/ur3e/physical_parameters.yaml'
+   visual_parameters_file:='$(find grinding_descriptions)/config/ur3e/visual_parameters.yaml'
    transmission_hw_interface:=hardware_interface/PositionJointInterface
    safety_limits:=false
@@ -29,5 +29,5 @@
    safety_k_position:=20"
   >
-    <xacro:include filename="$(find kek_scene_description)/urdf/inc/ur_macro.xacro" />
+    <xacro:include filename="$(find grinding_descriptions)/urdf/inc/ur_macro.xacro" />
     <xacro:ur_robot
       prefix="${prefix}"

File: catkin_ws/src/grinding_descriptions/urdf/inc/ur5_macro.xacro (robot description, xacro)
@@ -3,7 +3,7 @@
   <!--
     Convenience wrapper for the 'ur_robot' macro which provides default values
-    for the various "parameters files" parameters for a UR10.
+    for the various "parameters files" parameters for a UR5.
     This file can be used when composing a more complex scene with one or more
-    UR10 robots.
+    UR5 robots.
     While the generic 'ur_robot' macro could also be used, it would require
     the user to provide values for all parameters, as that macro does not set
@@ -17,11 +17,11 @@
           real robot.
   -->
-  <xacro:macro name="ur10_robot"
+  <xacro:macro name="ur5_robot"
     params="
    prefix
-   joint_limits_parameters_file:='$(find kek_scene_description)/config/ur10/joint_limits.yaml'
-   kinematics_parameters_file:='$(find kek_scene_description)/config/ur10/default_kinematics.yaml'
-   physical_parameters_file:='$(find kek_scene_description)/config/ur10/physical_parameters.yaml'
-   visual_parameters_file:='$(find kek_scene_description)/config/ur10/visual_parameters.yaml'
+   joint_limits_parameters_file:='$(find grinding_descriptions)/config/ur5/joint_limits.yaml'
+   kinematics_parameters_file:='$(find grinding_descriptions)/config/ur5/default_kinematics.yaml'
+   physical_parameters_file:='$(find grinding_descriptions)/config/ur5/physical_parameters.yaml'
+   visual_parameters_file:='$(find grinding_descriptions)/config/ur5/visual_parameters.yaml'
    transmission_hw_interface:=hardware_interface/PositionJointInterface
    safety_limits:=false
@@ -29,5 +29,5 @@
    safety_k_position:=20"
   >
-    <xacro:include filename="$(find kek_scene_description)/urdf/inc/ur_macro.xacro" />
+    <xacro:include filename="$(find grinding_descriptions)/urdf/inc/ur_macro.xacro" />
     <xacro:ur_robot
       prefix="${prefix}"

File: catkin_ws/src/grinding_descriptions/urdf/inc/ur5e_macro.xacro (robot description, xacro)
@@ -3,7 +3,7 @@
   <!--
     Convenience wrapper for the 'ur_robot' macro which provides default values
-    for the various "parameters files" parameters for a UR10e.
+    for the various "parameters files" parameters for a UR5e.
     This file can be used when composing a more complex scene with one or more
-    UR10e robots.
+    UR5e robots.
     While the generic 'ur_robot' macro could also be used, it would require
     the user to provide values for all parameters, as that macro does not set
@@ -17,11 +17,11 @@
           real robot.
   -->
-  <xacro:macro name="ur10e_robot"
+  <xacro:macro name="ur5e_robot"
     params="
    prefix
-   joint_limits_parameters_file:='$(find kek_scene_description)/config/ur10e/joint_limits.yaml'
-   kinematics_parameters_file:='$(find kek_scene_description)/config/ur10e/default_kinematics.yaml'
-   physical_parameters_file:='$(find kek_scene_description)/config/ur10e/physical_parameters.yaml'
-   visual_parameters_file:='$(find kek_scene_description)/config/ur10e/visual_parameters.yaml'
+   joint_limits_parameters_file:='$(find grinding_descriptions)/config/ur5e/joint_limits.yaml'
+   kinematics_parameters_file:='$(find grinding_descriptions)/config/ur5e/default_kinematics.yaml'
+   physical_parameters_file:='$(find grinding_descriptions)/config/ur5e/physical_parameters.yaml'
+   visual_parameters_file:='$(find grinding_descriptions)/config/ur5e/visual_parameters.yaml'
    transmission_hw_interface:=hardware_interface/PositionJointInterface
    safety_limits:=false
@@ -29,5 +29,5 @@
    safety_k_position:=20"
   >
-    <xacro:include filename="$(find kek_scene_description)/urdf/inc/ur_macro.xacro" />
+    <xacro:include filename="$(find grinding_descriptions)/urdf/inc/ur_macro.xacro" />
     <xacro:ur_robot
       prefix="${prefix}"

File: catkin_ws/src/grinding_descriptions/urdf/inc/ur_common.xacro (robot description, xacro)
@@ -22,5 +22,5 @@
           However, users MUST NOT rely on these properties, their contents or
           their names.
-          This macro is NOT part of the public API of the kek_scene_description pkg,
+          This macro is NOT part of the public API of the grinding_descriptions pkg,
           and as such should be considered to be for internal use only.
   -->

File: catkin_ws/src/grinding_descriptions/urdf/inc/ur_macro.xacro (robot description, xacro)
@@ -42,6 +42,6 @@
      - Muhammad Asif Rana
   -->
-  <xacro:include filename="$(find kek_scene_description)/urdf/inc/ur_transmissions.xacro" />
-  <xacro:include filename="$(find kek_scene_description)/urdf/inc/ur_common.xacro" />
+  <xacro:include filename="$(find grinding_descriptions)/urdf/inc/ur_transmissions.xacro" />
+  <xacro:include filename="$(find grinding_descriptions)/urdf/inc/ur_common.xacro" />
   <xacro:macro name="ur_robot"
     params="
@@ -222,5 +222,5 @@
         <geometry>
           <mesh
-            filename="package://kek_scene_description/mesh/Rviz/jig_pestle_spatula_spoon_UR5e.stl" />
+            filename="package://grinding_descriptions/mesh/Rviz/jig_pestle_spatula_spoon_UR5e.stl" />
         </geometry>
       </visual>
@@ -229,5 +229,5 @@
         <geometry>
           <mesh
-            filename="package://kek_scene_description/mesh/Rviz/jig_pestle_spatula_spoon_UR5e.stl" />
+            filename="package://grinding_descriptions/mesh/Rviz/jig_pestle_spatula_spoon_UR5e.stl" />
         </geometry>
       </collision>
@@ -246,5 +246,5 @@
         <geometry>
           <box size="0 0 0" />
-          <!-- <mesh filename="package://kek_scene_description/mesh/spatula_short_for_Rviz.stl" /> -->
+          <!-- <mesh filename="package://grinding_descriptions/mesh/spatula_short_for_Rviz.stl" /> -->
         </geometry>
       </visual>
@@ -254,5 +254,5 @@
         <origin xyz="0 0 0" rpy="0 0 0" />
         <geometry>
-          <mesh filename="package://kek_scene_description/mesh/spatula_short_for_Rviz.stl" />
+          <mesh filename="package://grinding_descriptions/mesh/spatula_short_for_Rviz.stl" />
         </geometry>
       </collision> -->
@@ -271,5 +271,5 @@
         <geometry>
           <box size="0 0 0" />
-          <!-- <mesh filename="package://kek_scene_description/mesh/spatula_short_for_Rviz.stl" /> -->
+          <!-- <mesh filename="package://grinding_descriptions/mesh/spatula_short_for_Rviz.stl" /> -->
         </geometry>
       </visual>
@@ -279,5 +279,5 @@
         <origin xyz="0 0 0" rpy="0 0 0" />
         <geometry>
-          <mesh filename="package://kek_scene_description/mesh/spatula_short_for_Rviz.stl" />
+          <mesh filename="package://grinding_descriptions/mesh/spatula_short_for_Rviz.stl" />
         </geometry>
       </collision> -->

File: catkin_ws/src/grinding_descriptions/urdf/pestle.urdf (robot description, URDF)
Before this commit: robot pestle, 2 links, 1 joints
Links:
- link pestle_link: geometry visual mesh filename=package://grinding_descriptions/mesh/jig_pestle_140.stl

File: catkin_ws/src/grinding_descriptions/urdf/pestle.urdf.xacro (robot description, xacro)
@@ -1,4 +1,4 @@
 <robot name="pestle"  xmlns:xacro="http://ros.org/wiki/xacro">
-  <xacro:property name="stl_file_path" value="package://kek_scene_description/mesh/jig_pestle_140.stl" />
+  <xacro:property name="stl_file_path" value="package://grinding_descriptions/mesh/jig_pestle_140.stl" />
   <link name="base_link"/>
   <joint name="pestle_joint" type="fixed">

File: catkin_ws/src/grinding_descriptions/urdf/ur.xacro (robot description, xacro)
@@ -2,5 +2,5 @@
 <robot xmlns:xacro="http://wiki.ros.org/xacro" name="ur">
       <!-- import main macro -->
-      <xacro:include filename="$(find kek_scene_description)/urdf/inc/ur_macro.xacro" />
+      <xacro:include filename="$(find grinding_descriptions)/urdf/inc/ur_macro.xacro" />
       <!-- parameters -->
       <xacro:arg name="joint_limit_params" default="" />

File: catkin_ws/src/grinding_descriptions/urdf/ur5e.xacro (robot description, xacro)
@@ -14,5 +14,5 @@
     Refer to 'inc/ur_macro.xacro' for more information.
   -->
-  <xacro:include filename="$(find kek_scene_description)/urdf/inc/ur5e_macro.xacro" />
+  <xacro:include filename="$(find grinding_descriptions)/urdf/inc/ur5e_macro.xacro" />
   <xacro:ur5e_robot prefix="" />
 </robot>

File: catkin_ws/src/grinding_descriptions/urdf/ur_macro.xacro (robot description, xacro)
@@ -42,6 +42,6 @@
      - Muhammad Asif Rana
   -->
-  <xacro:include filename="$(find kek_scene_description)/urdf/inc/ur_transmissions.xacro" />
-  <xacro:include filename="$(find kek_scene_description)/urdf/inc/ur_common.xacro" />
+  <xacro:include filename="$(find grinding_descriptions)/urdf/inc/ur_transmissions.xacro" />
+  <xacro:include filename="$(find grinding_descriptions)/urdf/inc/ur_common.xacro" />
   <xacro:macro name="ur_robot"
     params="
@@ -220,11 +220,11 @@
         <origin xyz="0 0 0" rpy="0 0 0" />
         <geometry>
-          <mesh filename="package://kek_scene_description/mesh/pestle_for_UR5e_without_spatula.stl" />
-        </geometry>
-      </visual>
-      <collision>
-        <origin xyz="0 0 0" rpy="0 0 0" />
-        <geometry>
-          <mesh filename="package://kek_scene_description/mesh/collision_jig_for_UR5e.stl" />
+          <mesh filename="package://grinding_descriptions/mesh/pestle_for_UR5e_without_spatula.stl" />
+        </geometry>
+      </visual>
+      <collision>
+        <origin xyz="0 0 0" rpy="0 0 0" />
+        <geometry>
+          <mesh filename="package://grinding_descriptions/mesh/collision_jig_for_UR5e.stl" />
         </geometry>
       </collision>
@@ -242,6 +242,6 @@
         <origin xyz="0 0 0" rpy="0 0 0" />
         <geometry>
-          <!-- <mesh filename="package://kek_scene_description/mesh/jig_spatula.stl"/> -->
-          <mesh filename="package://kek_scene_description/mesh/spatula_short_for_Rviz.stl" />
+          <!-- <mesh filename="package://grinding_descriptions/mesh/jig_spatula.stl"/> -->
+          <mesh filename="package://grinding_descriptions/mesh/spatula_short_for_Rviz.stl" />
         </geometry>
       </visual>
@@ -249,5 +249,5 @@
         <origin xyz="0 0 0" rpy="0 0 0"/>
         <geometry>
-          <mesh filename="package://kek_scene_description/mesh/jig_spatula.stl"/>
+          <mesh filename="package://grinding_descriptions/mesh/jig_spatula.stl"/>
         </geometry>
       </collision> -->
