Commit message: Add cobotta demo

File: catkin_ws/src/grinding_descriptions/urdf/cobotta/cobotta.urdf (robot description, URDF)
Before this commit: robot cobotta, 8 links, 7 joints
Links:
- added link pestle; visual mesh filename=package://grinding_descriptions/mesh/cobotta/jig_pestle_140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
- added link pestle_tip; visual box size=0 0 0
- added link spatula; visual mesh filename=package://grinding_descriptions/mesh/cobotta/jig_spatula.stl
- added link spatula_tip; visual box size=0 0 0
Joints:
- added joint joint_pestle: type fixed, parent J6, child pestle, origin xyz=0 0 0 rpy=0 0 0
- added joint joint_pestle_tip: type fixed, parent pestle, child pestle_tip, origin xyz=0 0 0.140 rpy=0 0 0
- added joint joint_spatula: type fixed, parent J6, child spatula, origin xyz=0 -0.026 0.049 rpy=0 0 -1.57079632679
- added joint joint_spatula_tip: type fixed, parent spatula, child spatula_tip, origin xyz=0.09 0 0 rpy=-1.57079632679 0 -1.57079632679

Commit message: Update cobotta demo params

File: catkin_ws/src/grinding_descriptions/urdf/cobotta/cobotta.urdf (robot description, URDF)
Before this commit: robot cobotta, 12 links, 11 joints
Joints:
- joint joint_pestle_tip: origin xyz=0 0 0.140 rpy=0 0 0 -> xyz=0 0 0.160 rpy=0 0 0

Commit message: Update cobotta 3D model

File: catkin_ws/src/grinding_descriptions/urdf/cobotta/cobotta.urdf (robot description, URDF)
Before this commit: robot cobotta, 12 links, 11 joints
Links:
- removed link pestle
- removed link pestle_tip
- removed link spatula
- removed link spatula_tip
- link J1: geometry collision mesh filename=package://grinding_descriptions/urdf/cobotta/J1.stl scale=1 1 1; visual mesh filename=package://grinding_descriptions/urdf/cobotta/J1.stl scale=1 1 1
- link J2: geometry collision mesh filename=package://grinding_descriptions/urdf/cobotta/J2.stl scale=1 1 1; visual mesh filename=package://grinding_descriptions/urdf/cobotta/J2.stl scale=1 1 1
- link J3: geometry collision mesh filename=package://grinding_descriptions/urdf/cobotta/J3.stl scale=1 1 1; visual mesh filename=package://grinding_descriptions/urdf/cobotta/J3.stl scale=1 1 1
- link J4: geometry collision mesh filename=package://grinding_descriptions/urdf/cobotta/J4.stl scale=1 1 1; visual mesh filename=package://grinding_descriptions/urdf/cobotta/J4.stl scale=1 1 1
- link J5: geometry collision mesh filename=package://grinding_descriptions/urdf/cobotta/J5.stl scale=1 1 1; visual mesh filename=package://grinding_descriptions/urdf/cobotta/J5.stl scale=1 1 1
- link J6: geometry collision mesh filename=package://grinding_descriptions/urdf/cobotta/J6.stl scale=1 1 1; visual mesh filename=package://grinding_descriptions/urdf/cobotta/J6.stl scale=1 1 1
- link base_link: geometry collision mesh filename=package://grinding_descriptions/urdf/cobotta/base_link.stl scale=1 1 1; visual mesh filename=package://grinding_descriptions/urdf/cobotta/base_link.stl scale=1 1 1
Joints:
- removed joint joint_pestle
- removed joint joint_pestle_tip
- removed joint joint_spatula
- removed joint joint_spatula_tip
- joint joint_1: limit lower=-2.61799387799149 upper=2.61799387799149 effort=1 velocity=0.383012504350156 -> lower=-2.617994 upper=2.617994 effort=1 velocity=0.383012504350156; origin xyz=0.000000 0.000000 0.000000 rpy=0.000000 0.000000 0.000000 -> xyz=0.000000 0.000000 0.108000 rpy=0.000000 0.000000 0.000000
- joint joint_2: limit lower=-1.0471975511966 upper=1.74532925199433 effort=1 velocity=0.37256670877697 -> lower=-1.047198 upper=1.745329 effort=1 velocity=0.37256670877697; origin xyz=0.000000 0.000000 0.180000 rpy=0.000000 0.000000 0.000000 -> xyz=0.000000 0.000000 0.072000 rpy=0.000000 0.000000 0.000000
- joint joint_3: limit lower=0.314159265358979 upper=2.44346095279206 effort=1 velocity=0.68942250783028 -> lower=0.3141593 upper=2.443461 effort=1 velocity=0.68942250783028
- joint joint_4: limit lower=-2.96705972839036 upper=2.96705972839036 effort=1 velocity=0.702189591308619 -> lower=-2.96706 upper=2.96706 effort=1 velocity=0.702189591308619; origin xyz=-0.012000 0.020000 -0.345000 rpy=0.000000 0.000000 0.000000 -> xyz=-0.012000 0.020000 0.088000 rpy=0.000000 0.000000 0.000000
- joint joint_5: limit lower=-1.65806278939461 upper=2.35619449019234 effort=1 velocity=0.702189591308619 -> lower=-1.658063 upper=2.356194 effort=1 velocity=0.702189591308619; origin xyz=0.000000 -0.020000 0.522500 rpy=0.000000 0.000000 0.000000 -> xyz=0.000000 -0.020000 0.089500 rpy=0.000000 0.000000 0.000000
- joint joint_6: limit lower=-2.96705972839036 upper=2.96705972839036 effort=1 velocity=1.05386470893922 -> lower=-2.96706 upper=2.96706 effort=1 velocity=1.05386470893922

Commit message: Add end effector

File: catkin_ws/src/grinding_descriptions/urdf/cobotta/cobotta.urdf (robot description, URDF)
Before this commit: robot cobotta, 8 links, 7 joints
Links:
- added link pestle; visual mesh filename=package://grinding_descriptions/mesh/cobotta/jig_pestle_140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
- added link pestle_tip; visual box size=0 0 0
- added link spatula; visual mesh filename=package://grinding_descriptions/mesh/cobotta/jig_spatula.stl
- added link spatula_tip; visual box size=0 0 0
Joints:
- added joint joint_pestle: type fixed, parent J6, child pestle, origin xyz=0 0 0 rpy=0 0 0
- added joint joint_pestle_tip: type fixed, parent pestle, child pestle_tip, origin xyz=0 0 0.160 rpy=0 0 0
- added joint joint_spatula: type fixed, parent J6, child spatula, origin xyz=0 -0.026 0.049 rpy=0 0 -1.57079632679
- added joint joint_spatula_tip: type fixed, parent spatula, child spatula_tip, origin xyz=0.09 0 0 rpy=-1.57079632679 0 -1.57079632679
