Commit message: Update URDF

File: catkin_ws/src/grinding_descriptions/urdf/ur5e/inc/ur_macro.xacro (robot description, xacro)
@@ -438,5 +438,5 @@
     </joint> -->
     <joint name="joint_spatula" type="fixed">
-      <origin rpy="0 ${-pi/2} 0" xyz="-0.03655 0 0.013" />
+      <origin rpy="0 ${-pi/2} 0" xyz="-0.03655 0 0.0135" />
       <parent link="${prefix}wrist_3_link" />
       <child link="spatula" />
@@ -449,5 +449,5 @@
     <!-- center of surface  on jig-->
     <joint name="joint_spoon" type="fixed">
-      <origin rpy="${-pi/2} 0 0" xyz="0.0075 0.042 0" />
+      <origin rpy="${-pi/2} 0 0" xyz="0.008 0.042 0" />
       <parent link="${prefix}flange" />
       <child link="spoon" />

Commit message: Add camera model

File: catkin_ws/src/grinding_descriptions/urdf/ur5e/inc/ur_macro.xacro (robot description, xacro)
@@ -215,5 +215,5 @@
       </xacro:cylinder_inertial>
     </link>
-    <!-- user (nakajima) added urdf for pestle -->
+    <!-- user (nakajima) added links -->
     <link name="pestle">
       <!-- 0.0001 means avoiding collision between pestle and wrist3 -->
@@ -290,4 +290,21 @@
         </geometry>
       </visual>
+    </link>
+    <link name="camera">
+      <!-- 0.0001 means avoiding collision between pestle and wrist3 -->
+      <visual>
+        <origin xyz="0 0 0.0001" rpy="0 0 0" />
+        <geometry>
+          <mesh
+            filename="package://grinding_descriptions/mesh/Rviz/Intel_RealSense_Depth_Camera_D435_v3.stl" />
+        </geometry>
+      </visual>
+      <collision>
+        <origin xyz="0 0 0.0001" rpy="0 0 0" />
+        <geometry>
+          <mesh
+            filename="package://grinding_descriptions/mesh/Rviz/Intel_RealSense_Depth_Camera_D435_v3.stl" />
+        </geometry>
+      </collision>
     </link>
     <!-- joints: main serial chain -->
@@ -391,15 +408,4 @@
       </xacro:if>
       <dynamics damping="0" friction="0" />
-    </joint>
-    <!-- user (nakajima) added urdf for pestle -->
-    <joint name="joint_pestle" type="fixed">
-      <origin rpy="0 0 0" xyz="0 0 0" />
-      <parent link="${prefix}wrist_3_link" />
-      <child link="pestle" />
-    </joint>
-    <joint name="joint_pestle_tip" type="fixed">
-      <origin rpy="0 0 0" xyz="0 0 0.130" />
-      <parent link="pestle" />
-      <child link="pestle_tip" />
     </joint>
     <!-- ROS-Industrial 'base' frame: base_link to UR 'Base' Coordinates transform -->
@@ -430,11 +436,31 @@
       <child link="${prefix}tool0" />
     </joint>
+    <!-- User (nakajima) added tool frame -->
+    <link name="${prefix}tool1" />
+    <joint name="${prefix}flange-tool1" type="fixed">
+      <!-- default toolframe: X+ left, Y+ up, Z+ front -->
+      <origin xyz="0.0075 0 0.0432" rpy="0 0 ${pi/2.0}" />
+      <parent link="${prefix}flange" />
+      <child link="${prefix}tool1" />
+    </joint>
+    <link name="${prefix}tool2" />
+    <joint name="${prefix}flange-tool2" type="fixed">
+      <!-- default toolframe: X+ left, Y+ up, Z+ front -->
+      <origin xyz="0.0075 0 -0.0432" rpy="0 ${pi} ${pi/2.0}" />
+      <parent link="${prefix}flange" />
+      <child link="${prefix}tool2" />
+    </joint>
+    <!-- user (nakajima) added joints -->
+    <joint name="joint_pestle" type="fixed">
+      <origin rpy="0 0 0" xyz="0 0 0" />
+      <parent link="${prefix}wrist_3_link" />
+      <child link="pestle" />
+    </joint>
+    <joint name="joint_pestle_tip" type="fixed">
+      <origin rpy="0 0 0" xyz="0 0 0.130" />
+      <parent link="pestle" />
+      <child link="pestle_tip" />
+    </joint>
     <!-- center of surface on spatula bearing -->
-    <!-- twist3はrevolteし解が定まらないのでfixedされているflangeのjointをparentにする -->
-    <!-- <joint name="joint_spatula" type="fixed">
-      <origin rpy="${pi/2} 0 0" xyz="0.013 -0.03655 0" />
-      <parent link="${prefix}flange" />
-      <child link="spatula" />
-    </joint> -->
     <joint name="joint_spatula" type="fixed">
       <origin rpy="0 ${-pi/2} 0" xyz="-0.03655 0 0.013" />
@@ -454,9 +480,13 @@
     </joint>
     <joint name="joint_spoon_tip" type="fixed">
-      <!-- <origin rpy="0 0 0" xyz="0.03 0 0.115" /> -->
       <origin rpy="0 0 0" xyz="0.02 0 0.115" />
       <parent link="spoon" />
       <child link="spoon_tip" />
     </joint>
+    <joint name="joint_camera" type="fixed">
+      <origin rpy="0 0 ${-pi/2.0}" xyz="0 0.0605 0.03" />
+      <parent link="${prefix}tool2" />
+      <child link="camera" />
+    </joint>
   </xacro:macro>
 </robot>

Commit message: Update URDF

File: catkin_ws/src/grinding_descriptions/urdf/ur5e/inc/ur_macro.xacro (robot description, xacro)
@@ -291,5 +291,5 @@
       </visual>
     </link>
-    <link name="camera">
+    <link name="camera_jig">
       <!-- 0.0001 means avoiding collision between pestle and wrist3 -->
       <visual>
@@ -307,4 +307,12 @@
         </geometry>
       </collision>
+    </link>
+    <link name="calibrated_color_optical_frame">
+      <visual>
+        <origin xyz="0 0 0" rpy="0 0 0" />
+        <geometry>
+          <box size="0 0 0" />
+        </geometry>
+      </visual>
     </link>
     <!-- joints: main serial chain -->
@@ -484,8 +492,14 @@
       <child link="spoon_tip" />
     </joint>
-    <joint name="joint_camera" type="fixed">
+    <joint name="joint_camera_jig" type="fixed">
       <origin rpy="0 0 ${-pi/2.0}" xyz="0 0.0605 0.03" />
       <parent link="${prefix}tool2" />
-      <child link="camera" />
+      <child link="camera_jig" />
+    </joint>
+    <!-- This frame is calculated by MoveitCalibration -->
+    <joint name="joint_calibrated_color_optical_frame" type="fixed">
+      <origin rpy="1.5208 0.0225205 -1.57642" xyz="0.0016629 -0.0548537 -0.0260291" />
+      <parent link="${prefix}tool0" />
+      <child link="calibrated_color_optical_frame" />
     </joint>
   </xacro:macro>

Commit message: Add optical frame

File: catkin_ws/src/grinding_descriptions/urdf/ur5e/inc/ur_macro.xacro (robot description, xacro)
@@ -316,4 +316,12 @@
       </visual>
     </link>
+    <link name="calibrated_depth_optical_frame">
+      <visual>
+        <origin xyz="0 0 0" rpy="0 0 0" />
+        <geometry>
+          <box size="0 0 0" />
+        </geometry>
+      </visual>
+    </link>
     <!-- joints: main serial chain -->
     <joint name="${prefix}base_link-base_link_inertia" type="fixed">
@@ -503,4 +511,9 @@
       <child link="calibrated_color_optical_frame" />
     </joint>
+    <joint name="joint_calibrated_depth_optical_frame" type="fixed">
+      <origin rpy="${-pi/2} 0 ${-pi/2}" xyz="0 0 0" />
+      <parent link="calibrated_color_optical_frame" />
+      <child link="calibrated_depth_optical_frame" />
+    </joint>
   </xacro:macro>
 </robot>

Commit message: Update estimated mortar position by vision

File: catkin_ws/src/grinding_descriptions/urdf/ur5e/inc/ur_macro.xacro (robot description, xacro)
@@ -507,10 +507,10 @@
     <!-- This frame is calculated by MoveitCalibration -->
     <joint name="joint_calibrated_color_optical_frame" type="fixed">
-      <origin rpy="1.5208 0.0225205 -1.57642" xyz="0.0016629 -0.0548537 -0.0260291" />
-      <parent link="${prefix}tool0" />
+      <origin xyz="-0.0147918 -0.000782691 -0.050422" rpy="0.0053461 3.11399 0.0150722" />
+      <parent link="${prefix}flange" />
       <child link="calibrated_color_optical_frame" />
     </joint>
     <joint name="joint_calibrated_depth_optical_frame" type="fixed">
-      <origin rpy="${-pi/2} 0 ${-pi/2}" xyz="0 0 0" />
+      <origin rpy="0 0 0" xyz="0 0 0" />
       <parent link="calibrated_color_optical_frame" />
       <child link="calibrated_depth_optical_frame" />

Commit message: Update URDF

File: catkin_ws/src/grinding_descriptions/urdf/ur5e/inc/ur_macro.xacro (robot description, xacro)
@@ -291,21 +291,4 @@
       </visual>
     </link>
-    <link name="camera_jig">
-      <!-- 0.0001 means avoiding collision between pestle and wrist3 -->
-      <visual>
-        <origin xyz="0 0 0.0001" rpy="0 0 0" />
-        <geometry>
-          <mesh
-            filename="package://grinding_descriptions/mesh/Rviz/Intel_RealSense_Depth_Camera_D435_v3.stl" />
-        </geometry>
-      </visual>
-      <collision>
-        <origin xyz="0 0 0.0001" rpy="0 0 0" />
-        <geometry>
-          <mesh
-            filename="package://grinding_descriptions/mesh/Rviz/Intel_RealSense_Depth_Camera_D435_v3.stl" />
-        </geometry>
-      </collision>
-    </link>
     <link name="calibrated_color_optical_frame">
       <visual>
@@ -463,7 +446,14 @@
     <joint name="${prefix}flange-tool2" type="fixed">
       <!-- default toolframe: X+ left, Y+ up, Z+ front -->
+      <origin xyz="0.0075 0.0432 0" rpy="${-pi/2.0} ${pi/2.0} 0" />
+      <parent link="${prefix}flange" />
+      <child link="${prefix}tool2" />
+    </joint>
+    <link name="${prefix}tool3" />
+    <joint name="${prefix}flange-tool3" type="fixed">
+      <!-- default toolframe: X+ left, Y+ up, Z+ front -->
       <origin xyz="0.0075 0 -0.0432" rpy="0 ${pi} ${pi/2.0}" />
       <parent link="${prefix}flange" />
-      <child link="${prefix}tool2" />
+      <child link="${prefix}tool3" />
     </joint>
     <!-- user (nakajima) added joints -->
@@ -474,10 +464,10 @@
     </joint>
     <joint name="joint_pestle_tip" type="fixed">
-      <origin rpy="0 0 0" xyz="0 0 0.130" />
+      <origin rpy="0 0 0" xyz="0 0 0.12044162537801482" />
       <parent link="pestle" />
       <child link="pestle_tip" />
     </joint>
     <!-- center of surface on spatula bearing -->
-    <joint name="joint_spatula" type="fixed">
+    <!-- <joint name="joint_spatula" type="fixed">
       <origin rpy="0 ${-pi/2} 0" xyz="-0.03655 0 0.0135" />
       <parent link="${prefix}wrist_3_link" />
@@ -488,21 +478,31 @@
       <parent link="spatula" />
       <child link="spatula_tip" />
+    </joint> -->
+    <joint name="joint_spatula" type="fixed">
+      <origin rpy="0 0 0" xyz="0 0 0" />
+      <parent link="${prefix}tool1" />
+      <child link="spatula" />
+    </joint>
+    <joint name="joint_spatula_tip" type="fixed">
+      <origin rpy="0 0 0" xyz="0 0 0.092" />
+      <parent link="spatula" />
+      <child link="spatula_tip" />
     </joint>
     <!-- center of surface  on jig-->
     <joint name="joint_spoon" type="fixed">
-      <origin rpy="${-pi/2} 0 0" xyz="0.008 0.042 0" />
-      <parent link="${prefix}flange" />
+      <origin rpy="0 0 0" xyz="0 0 0" />
+      <parent link="${prefix}tool2" />
       <child link="spoon" />
     </joint>
     <joint name="joint_spoon_tip" type="fixed">
-      <origin rpy="0 0 0" xyz="0.02 0 0.115" />
+      <origin rpy="0 0 ${pi}" xyz="0 -0.025 0.145" />
       <parent link="spoon" />
       <child link="spoon_tip" />
     </joint>
-    <joint name="joint_camera_jig" type="fixed">
+    <!-- <joint name="joint_camera_jig" type="fixed">
       <origin rpy="0 0 ${-pi/2.0}" xyz="0 0.0605 0.03" />
-      <parent link="${prefix}tool2" />
+      <parent link="${prefix}tool3" />
       <child link="camera_jig" />
-    </joint>
+    </joint> -->
     <!-- This frame is calculated by MoveitCalibration -->
     <joint name="joint_calibrated_color_optical_frame" type="fixed">

Commit message: Add calibrated mortar pos

File: catkin_ws/src/grinding_descriptions/urdf/ur5e/inc/ur_macro.xacro (robot description, xacro)
@@ -464,5 +464,5 @@
     </joint>
     <joint name="joint_pestle_tip" type="fixed">
-      <origin rpy="0 0 0" xyz="0 0 0.12044162537801482" />
+      <origin rpy="0 0 0" xyz="0 0 0.12325432750182237" />
       <parent link="pestle" />
       <child link="pestle_tip" />

Commit message: Update params

File: catkin_ws/src/grinding_descriptions/urdf/ur5e/inc/ur_macro.xacro (robot description, xacro)
@@ -469,7 +469,17 @@
     </joint>
     <!-- center of surface on spatula bearing -->
-    <!-- <joint name="joint_spatula" type="fixed">
+    <joint name="joint_spatula" type="fixed">
       <origin rpy="0 ${-pi/2} 0" xyz="-0.03655 0 0.0135" />
       <parent link="${prefix}wrist_3_link" />
+      <child link="spatula" />
+    </joint>
+    <joint name="joint_spatula_tip" type="fixed">
+      <origin rpy="0 0 0" xyz="0 0 0.092" />
+      <parent link="spatula" />
+      <child link="spatula_tip" />
+    </joint>
+    <!-- <joint name="joint_spatula" type="fixed">
+      <origin rpy="0 0 0" xyz="0 0 0" />
+      <parent link="${prefix}tool1" />
       <child link="spatula" />
     </joint>
@@ -479,14 +489,4 @@
       <child link="spatula_tip" />
     </joint> -->
-    <joint name="joint_spatula" type="fixed">
-      <origin rpy="0 0 0" xyz="0 0 0" />
-      <parent link="${prefix}tool1" />
-      <child link="spatula" />
-    </joint>
-    <joint name="joint_spatula_tip" type="fixed">
-      <origin rpy="0 0 0" xyz="0 0 0.092" />
-      <parent link="spatula" />
-      <child link="spatula_tip" />
-    </joint>
     <!-- center of surface  on jig-->
     <joint name="joint_spoon" type="fixed">

Commit message: Update URDF

File: catkin_ws/src/grinding_descriptions/urdf/ur5e/inc/ur_macro.xacro (robot description, xacro)
@@ -464,5 +464,5 @@
     </joint>
     <joint name="joint_pestle_tip" type="fixed">
-      <origin rpy="0 0 0" xyz="0 0 0.12325432750182237" />
+      <origin rpy="0 0 0" xyz="0 0 0.12324" />
       <parent link="pestle" />
       <child link="pestle_tip" />
