Commit message: Update URDF

File: catkin_ws/src/grinding_descriptions/urdf/ur/inc/ur_macro.xacro (robot description, xacro)
@@ -222,5 +222,5 @@
         <geometry>
           <mesh
-            filename="package://grinding_descriptions/mesh/Rviz/jig_pestle_spatula_spoon_UR5e.stl" />
+            filename="package://grinding_descriptions/mesh/end_effector/pestle_ur.stl" />
         </geometry>
       </visual>
@@ -229,5 +229,5 @@
         <geometry>
           <mesh
-            filename="package://grinding_descriptions/mesh/Rviz/jig_pestle_spatula_spoon_UR5e.stl" />
+            filename="package://grinding_descriptions/mesh/end_effector/pestle_ur.stl" />
         </geometry>
       </collision>
@@ -243,18 +243,15 @@
     <link name="spatula">
       <visual>
-        <origin xyz="0 0 0" rpy="0 0 0" />
-        <geometry>
-          <box size="0 0 0" />
-          <!-- <mesh filename="package://grinding_descriptions/mesh/spatula_short_for_Rviz.stl" /> -->
-        </geometry>
-      </visual>
-      <!-- comment out collision because to avoid collision check between spatula and pestle in
-      MoveIt -->
-      <!-- <collision>
-        <origin xyz="0 0 0" rpy="0 0 0" />
-        <geometry>
-          <mesh filename="package://grinding_descriptions/mesh/spatula_short_for_Rviz.stl" />
-        </geometry>
-      </collision> -->
+        <origin xyz="0 0 0.0001" rpy="0 0 0" />
+        <geometry>
+          <mesh filename="package://grinding_descriptions/mesh/end_effector/spatula.stl" />
+        </geometry>
+      </visual>
+      <collision>
+        <origin xyz="0 0 0.0001" rpy="0 0 0" />
+        <geometry>
+          <mesh filename="package://grinding_descriptions/mesh/end_effector/spatula.stl" />
+        </geometry>
+      </collision>
     </link>
     <link name="spatula_tip">
@@ -475,5 +472,5 @@
     </joint>
     <joint name="joint_spatula_tip" type="fixed">
-      <origin rpy="0 0 0" xyz="0 0 0.092" />
+      <origin rpy="0 0 0" xyz="0 0 0.081" />
       <parent link="spatula" />
       <child link="spatula_tip" />
