Commit message: Add xacro and create new urdf

File: grinding_descriptions/urdf/cobotta/setup_files/cobotta_description/cobotta.urdf (robot description, URDF)
Before this commit: robot cobotta, 12 links, 11 joints
Links:
- link J1: mass 1 -> 1.29
- link J2: mass 1 -> 0.39
- link J3: mass 1 -> 0.35
- link J4: mass 1 -> 0.35
- link J5: mass 1 -> 0.19
- link J6: mass 1 -> 0.03
- link base_link: mass 1 -> 1.4
