Commit message: Update dynamics params

File: grinding_descriptions/urdf/cobotta/setup_files/cobotta.urdf.xacro (robot description, xacro)
@@ -75,5 +75,5 @@
 		<axis xyz="-0.000000 -0.000000 1.000000" />
 		<limit effort="1" lower="-2.617994" upper="2.617994" velocity="0.383012504350156" />
-		<dynamics damping="0" friction="0" />
+		<dynamics damping="${joint_damping}" friction="${joint_friction}" />
 	</joint>
 	<transmission name="trans_1">
@@ -110,5 +110,5 @@
 		<axis xyz="-0.000000 1.000000 -0.000000" />
 		<limit effort="1" lower="-1.047198" upper="1.745329" velocity="0.37256670877697" />
-		<dynamics damping="0" friction="0" />
+		<dynamics damping="${joint_damping}" friction="${joint_friction}" />
 	</joint>
 	<transmission name="trans_2">
@@ -145,5 +145,5 @@
 		<axis xyz="-0.000000 1.000000 -0.000000" />
 		<limit effort="1" lower="0.3141593" upper="2.443461" velocity="0.68942250783028" />
-		<dynamics damping="0" friction="0" />
+		<dynamics damping="${joint_damping}" friction="${joint_friction}" />
 	</joint>
 	<transmission name="trans_3">
@@ -180,5 +180,5 @@
 		<axis xyz="-0.000000 -0.000000 1.000000" />
 		<limit effort="1" lower="-2.96706" upper="2.96706" velocity="0.702189591308619" />
-		<dynamics damping="0" friction="0" />
+		<dynamics damping="${joint_damping}" friction="${joint_friction}" />
 	</joint>
 	<transmission name="trans_4">
@@ -215,5 +215,5 @@
 		<axis xyz="-0.000000 1.000000 -0.000000" />
 		<limit effort="1" lower="-1.658063" upper="2.356194" velocity="0.702189591308619" />
-		<dynamics damping="0" friction="0" />
+		<dynamics damping="${joint_damping}" friction="${joint_friction}" />
 	</joint>
 	<transmission name="trans_5">
@@ -250,5 +250,5 @@
 		<axis xyz="-0.000000 -0.000000 1.000000" />
 		<limit effort="1" lower="-2.96706" upper="2.96706" velocity="1.05386470893922" />
-		<dynamics damping="0" friction="0" />
+		<dynamics damping="${joint_damping}" friction="${joint_friction}" />
 	</joint>
 	<transmission name="trans_6">

Commit message: Update

File: grinding_descriptions/urdf/cobotta/setup_files/cobotta.urdf.xacro (robot description, xacro)
@@ -37,5 +37,5 @@
 			<origin rpy="0 0 0" xyz="0 0 0" />
 			<geometry>
-				<mesh filename="package://grinding_descriptions/urdf/cobotta/base_link.stl"
+				<mesh filename="package://grinding_descriptions/urdf/cobotta/base_link.dae"
 					scale="1 1 1" />
 			</geometry>
@@ -44,5 +44,5 @@
 			<origin rpy="0 0 0" xyz="0 0 0" />
 			<geometry>
-				<mesh filename="package://grinding_descriptions/urdf/cobotta/base_link.stl"
+				<mesh filename="package://grinding_descriptions/urdf/cobotta/base_link.dae"
 					scale="1 1 1" />
 			</geometry>
@@ -56,11 +56,11 @@
 			<origin rpy="0 0 0" xyz="0 0 0" />
 			<geometry>
-				<mesh filename="package://grinding_descriptions/urdf/cobotta/J1.stl" scale="1 1 1" />
-			</geometry>
-		</visual>
-		<collision>
-			<origin rpy="0 0 0" xyz="0 0 0" />
-			<geometry>
-				<mesh filename="package://grinding_descriptions/urdf/cobotta/J1.stl" scale="1 1 1" />
+				<mesh filename="package://grinding_descriptions/urdf/cobotta/J1.dae" scale="1 1 1" />
+			</geometry>
+		</visual>
+		<collision>
+			<origin rpy="0 0 0" xyz="0 0 0" />
+			<geometry>
+				<mesh filename="package://grinding_descriptions/urdf/cobotta/J1.dae" scale="1 1 1" />
 			</geometry>
 		</collision>
@@ -72,7 +72,7 @@
 		<parent link="base_link" />
 		<child link="J1" />
-		<origin rpy="0.000000 0.000000 0.000000" xyz="0.000000 0.000000 0.108000" />
+		<origin rpy="0.000000 0.000000 0.000000" xyz="0.000000 0.000000 0.000000" />
 		<axis xyz="-0.000000 -0.000000 1.000000" />
-		<limit effort="1" lower="-2.617994" upper="2.617994" velocity="0.383012504350156" />
+		<limit effort="10" lower="-2.617994" upper="2.617994" velocity="0.383012504350156" />
 		<dynamics damping="${joint_damping}" friction="${joint_friction}" />
 	</joint>
@@ -91,11 +91,11 @@
 			<origin rpy="0 0 0" xyz="0 0 0" />
 			<geometry>
-				<mesh filename="package://grinding_descriptions/urdf/cobotta/J2.stl" scale="1 1 1" />
-			</geometry>
-		</visual>
-		<collision>
-			<origin rpy="0 0 0" xyz="0 0 0" />
-			<geometry>
-				<mesh filename="package://grinding_descriptions/urdf/cobotta/J2.stl" scale="1 1 1" />
+				<mesh filename="package://grinding_descriptions/urdf/cobotta/J2.dae" scale="1 1 1" />
+			</geometry>
+		</visual>
+		<collision>
+			<origin rpy="0 0 0" xyz="0 0 0" />
+			<geometry>
+				<mesh filename="package://grinding_descriptions/urdf/cobotta/J2.dae" scale="1 1 1" />
 			</geometry>
 		</collision>
@@ -109,5 +109,5 @@
 		<origin rpy="0.000000 0.000000 0.000000" xyz="0.000000 0.000000 0.072000" />
 		<axis xyz="-0.000000 1.000000 -0.000000" />
-		<limit effort="1" lower="-1.047198" upper="1.745329" velocity="0.37256670877697" />
+		<limit effort="10" lower="-1.047198" upper="1.745329" velocity="0.37256670877697" />
 		<dynamics damping="${joint_damping}" friction="${joint_friction}" />
 	</joint>
@@ -126,11 +126,11 @@
 			<origin rpy="0 0 0" xyz="0 0 0" />
 			<geometry>
-				<mesh filename="package://grinding_descriptions/urdf/cobotta/J3.stl" scale="1 1 1" />
-			</geometry>
-		</visual>
-		<collision>
-			<origin rpy="0 0 0" xyz="0 0 0" />
-			<geometry>
-				<mesh filename="package://grinding_descriptions/urdf/cobotta/J3.stl" scale="1 1 1" />
+				<mesh filename="package://grinding_descriptions/urdf/cobotta/J3.dae" scale="1 1 1" />
+			</geometry>
+		</visual>
+		<collision>
+			<origin rpy="0 0 0" xyz="0 0 0" />
+			<geometry>
+				<mesh filename="package://grinding_descriptions/urdf/cobotta/J3.dae" scale="1 1 1" />
 			</geometry>
 		</collision>
@@ -144,5 +144,5 @@
 		<origin rpy="0.000000 0.000000 0.000000" xyz="0.000000 0.000000 0.165000" />
 		<axis xyz="-0.000000 1.000000 -0.000000" />
-		<limit effort="1" lower="0.3141593" upper="2.443461" velocity="0.68942250783028" />
+		<limit effort="10" lower="0.3141593" upper="2.443461" velocity="0.68942250783028" />
 		<dynamics damping="${joint_damping}" friction="${joint_friction}" />
 	</joint>
@@ -161,11 +161,11 @@
 			<origin rpy="0 0 0" xyz="0 0 0" />
 			<geometry>
-				<mesh filename="package://grinding_descriptions/urdf/cobotta/J4.stl" scale="1 1 1" />
-			</geometry>
-		</visual>
-		<collision>
-			<origin rpy="0 0 0" xyz="0 0 0" />
-			<geometry>
-				<mesh filename="package://grinding_descriptions/urdf/cobotta/J4.stl" scale="1 1 1" />
+				<mesh filename="package://grinding_descriptions/urdf/cobotta/J4.dae" scale="1 1 1" />
+			</geometry>
+		</visual>
+		<collision>
+			<origin rpy="0 0 0" xyz="0 0 0" />
+			<geometry>
+				<mesh filename="package://grinding_descriptions/urdf/cobotta/J4.dae" scale="1 1 1" />
 			</geometry>
 		</collision>
@@ -179,5 +179,5 @@
 		<origin rpy="0.000000 0.000000 0.000000" xyz="-0.012000 0.020000 0.088000" />
 		<axis xyz="-0.000000 -0.000000 1.000000" />
-		<limit effort="1" lower="-2.96706" upper="2.96706" velocity="0.702189591308619" />
+		<limit effort="10" lower="-2.96706" upper="2.96706" velocity="0.702189591308619" />
 		<dynamics damping="${joint_damping}" friction="${joint_friction}" />
 	</joint>
@@ -196,11 +196,11 @@
 			<origin rpy="0 0 0" xyz="0 0 0" />
 			<geometry>
-				<mesh filename="package://grinding_descriptions/urdf/cobotta/J5.stl" scale="1 1 1" />
-			</geometry>
-		</visual>
-		<collision>
-			<origin rpy="0 0 0" xyz="0 0 0" />
-			<geometry>
-				<mesh filename="package://grinding_descriptions/urdf/cobotta/J5.stl" scale="1 1 1" />
+				<mesh filename="package://grinding_descriptions/urdf/cobotta/J5.dae" scale="1 1 1" />
+			</geometry>
+		</visual>
+		<collision>
+			<origin rpy="0 0 0" xyz="0 0 0" />
+			<geometry>
+				<mesh filename="package://grinding_descriptions/urdf/cobotta/J5.dae" scale="1 1 1" />
 			</geometry>
 		</collision>
@@ -214,5 +214,5 @@
 		<origin rpy="0.000000 0.000000 0.000000" xyz="0.000000 -0.020000 0.089500" />
 		<axis xyz="-0.000000 1.000000 -0.000000" />
-		<limit effort="1" lower="-1.658063" upper="2.356194" velocity="0.702189591308619" />
+		<limit effort="10" lower="-1.658063" upper="2.356194" velocity="0.702189591308619" />
 		<dynamics damping="${joint_damping}" friction="${joint_friction}" />
 	</joint>
@@ -231,11 +231,11 @@
 			<origin rpy="0 0 0" xyz="0 0 0" />
 			<geometry>
-				<mesh filename="package://grinding_descriptions/urdf/cobotta/J6.stl" scale="1 1 1" />
-			</geometry>
-		</visual>
-		<collision>
-			<origin rpy="0 0 0" xyz="0 0 0" />
-			<geometry>
-				<mesh filename="package://grinding_descriptions/urdf/cobotta/J6.stl" scale="1 1 1" />
+				<mesh filename="package://grinding_descriptions/urdf/cobotta/J6.dae" scale="1 1 1" />
+			</geometry>
+		</visual>
+		<collision>
+			<origin rpy="0 0 0" xyz="0 0 0" />
+			<geometry>
+				<mesh filename="package://grinding_descriptions/urdf/cobotta/J6.dae" scale="1 1 1" />
 			</geometry>
 		</collision>
@@ -249,5 +249,5 @@
 		<origin rpy="0.000000 0.000000 0.000000" xyz="0.000000 -0.044500 0.042000" />
 		<axis xyz="-0.000000 -0.000000 1.000000" />
-		<limit effort="1" lower="-2.96706" upper="2.96706" velocity="1.05386470893922" />
+		<limit effort="10" lower="-2.96706" upper="2.96706" velocity="1.05386470893922" />
 		<dynamics damping="${joint_damping}" friction="${joint_friction}" />
 	</joint>
@@ -290,17 +290,17 @@
 		<child link="spatula_tip" />
 	</joint>
-	<link name="pestle">
-		<visual>
-			<geometry>
-				<mesh filename="package://grinding_descriptions/mesh/cobotta/jig_pestle_140.stl" />
-			</geometry>
-		</visual>
-	</link>
-	<joint name="joint_pestle" type="fixed">
+	<link name="pedaee">
+		<visual>
+			<geometry>
+				<mesh filename="package://grinding_descriptions/mesh/cobotta/jig_pedaee_140.stl" />
+			</geometry>
+		</visual>
+	</link>
+	<joint name="joint_pedaee" type="fixed">
 		<origin rpy="0 0 0" xyz="0 0 0" />
 		<parent link="J6" />
-		<child link="pestle" />
-	</joint>
-	<link name="pestle_tip">
+		<child link="pedaee" />
+	</joint>
+	<link name="pedaee_tip">
 		<visual>
 			<geometry>
@@ -309,9 +309,9 @@
 		</visual>
 	</link>
-	<joint name="joint_pestle_tip" type="fixed">
-		<!-- for pestle -->
+	<joint name="joint_pedaee_tip" type="fixed">
+		<!-- for pedaee -->
 		<origin rpy="0 0 0" xyz="0 0 0.160" />
-		<parent link="pestle" />
-		<child link="pestle_tip" />
+		<parent link="pedaee" />
+		<child link="pedaee_tip" />
 	</joint>
 </robot>

Commit message: Fix name

File: grinding_descriptions/urdf/cobotta/setup_files/cobotta.urdf.xacro (robot description, xacro)
@@ -290,17 +290,17 @@
 		<child link="spatula_tip" />
 	</joint>
-	<link name="pedaee">
-		<visual>
-			<geometry>
-				<mesh filename="package://grinding_descriptions/mesh/cobotta/jig_pedaee_140.stl" />
-			</geometry>
-		</visual>
-	</link>
-	<joint name="joint_pedaee" type="fixed">
+	<link name="pestle">
+		<visual>
+			<geometry>
+				<mesh filename="package://grinding_descriptions/mesh/cobotta/jig_pestle_140.stl" />
+			</geometry>
+		</visual>
+	</link>
+	<joint name="joint_pestle" type="fixed">
 		<origin rpy="0 0 0" xyz="0 0 0" />
 		<parent link="J6" />
-		<child link="pedaee" />
-	</joint>
-	<link name="pedaee_tip">
+		<child link="pestle" />
+	</joint>
+	<link name="pestle_tip">
 		<visual>
 			<geometry>
@@ -309,9 +309,9 @@
 		</visual>
 	</link>
-	<joint name="joint_pedaee_tip" type="fixed">
-		<!-- for pedaee -->
+	<joint name="joint_pestle_tip" type="fixed">
+		<!-- for pestle -->
 		<origin rpy="0 0 0" xyz="0 0 0.160" />
-		<parent link="pedaee" />
-		<child link="pedaee_tip" />
+		<parent link="pestle" />
+		<child link="pestle_tip" />
 	</joint>
 </robot>
