Commit message: Update contol algorithm

File: grinding_descriptions/urdf/ur/inc/ur_macro.xacro (robot description, xacro)
@@ -461,5 +461,5 @@
     </joint>
     <joint name="joint_pestle_tip" type="fixed">
-      <origin rpy="0 0 0" xyz="0 0 0.12324" />
+      <origin rpy="0 0 0" xyz="0 0 0.12124" />
       <parent link="pestle" />
       <child link="pestle_tip" />
@@ -472,5 +472,5 @@
     </joint>
     <joint name="joint_spatula_tip" type="fixed">
-      <origin rpy="0 0 0" xyz="0 0 0.081" />
+      <origin rpy="0 0 0" xyz="0 0 0.091" />
       <parent link="spatula" />
       <child link="spatula_tip" />
