Commit message: Add end effector

File: grinding_descriptions/urdf/cobotta_pro_900/cobotta_pro_900.urdf (robot description, URDF)
Before this commit: robot cobotta_pro_900, 8 links, 7 joints
Links:
- added link flange
- added link pestle; collision mesh filename=package://grinding_descriptions/mesh/end_effector/pestle_ur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; visual mesh filename=package://grinding_descriptions/mesh/end_effector/pestle_ur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
- added link pestle_tip; visual box size=0 0 0
- added link spatula; collision mesh filename=package://grinding_descriptions/mesh/end_effector/spatula.s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; visual mesh filename=package://grinding_descriptions/mesh/end_effector/spatula.s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
- added link spatula_tip; visual box size=0 0 0
Joints:
- added joint joint_pestle: type fixed, parent flange, child pestle, origin xyz=0 0 0 rpy=0 0 0
- added joint joint_pestle_tip: type fixed, parent pestle, child pestle_tip, origin xyz=0 0 0.12324 rpy=0 0 0
- added joint joint_spatula: type fixed, parent flange, child spatula, origin xyz=-0.03655 0 0.0135 rpy=0 -1.570795 0
- added joint joint_spatula_tip: type fixed, parent spatula, child spatula_tip, origin xyz=0 0 0.081 rpy=0 0 0
- added joint wrist_3-flange: type fixed, parent J6, child flange, origin xyz=0 0 0 rpy=0 0 0

Commit message: Update mesh address

File: grinding_descriptions/urdf/cobotta_pro_900/cobotta_pro_900.urdf (robot description, URDF)
Before this commit: robot cobotta_pro_900, 13 links, 12 joints
Links:
- link J1: geometry collision mesh filename=package://grinding_descriptions/urdf/cobotta_pro_900/J1.dae scale=1 1 1; visual mesh filename=package://grinding_descriptions/urdf/cobotta_pro_900/J1.dae scale=1 1 1
- link J2: geometry collision mesh filename=package://grinding_descriptions/urdf/cobotta_pro_900/J2.dae scale=1 1 1; visual mesh filename=package://grinding_descriptions/urdf/cobotta_pro_900/J2.dae scale=1 1 1
- link J3: geometry collision mesh filename=package://grinding_descriptions/urdf/cobotta_pro_900/J3.dae scale=1 1 1; visual mesh filename=package://grinding_descriptions/urdf/cobotta_pro_900/J3.dae scale=1 1 1
- link J4: geometry collision mesh filename=package://grinding_descriptions/urdf/cobotta_pro_900/J4.dae scale=1 1 1; visual mesh filename=package://grinding_descriptions/urdf/cobotta_pro_900/J4.dae scale=1 1 1
- link J5: geometry collision mesh filename=package://grinding_descriptions/urdf/cobotta_pro_900/J5.dae scale=1 1 1; visual mesh filename=package://grinding_descriptions/urdf/cobotta_pro_900/J5.dae scale=1 1 1
- link J6: geometry collision mesh filename=package://grinding_descriptions/urdf/cobotta_pro_900/J6.dae scale=1 1 1; visual mesh filename=package://grinding_descriptions/urdf/cobotta_pro_900/J6.dae scale=1 1 1
- link base_link: geometry collision mesh filename=package://grinding_descriptions/urdf/cobotta_pro_900/base_l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 scale=1 1 1; visual mesh filename=package://grinding_descriptions/urdf/cobotta_pro_900/base_l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 scale=1 1 1

File: grinding_descriptions/urdf/fr3/fr3v5.urdf (robot description, URDF)
Before this commit: robot fr3v5, 13 links, 12 joints
Links:
- link base_link: geometry collision mesh filename=package://grinding_descriptions/meshes/fr3v5/collision/base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; visual mesh filename=package://grinding_descriptions/meshes/fr3v5/visual/base_li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
- link forearm_Link: geometry collision mesh filename=package://grinding_descriptions/meshes/fr3v5/collision/fore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; visual mesh filename=package://grinding_descriptions/meshes/fr3v5/visual/forearm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
- link shoulder_Link: geometry collision mesh filename=package://grinding_descriptions/meshes/fr3v5/collision/shou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; visual mesh filename=package://grinding_descriptions/meshes/fr3v5/visual/shoulde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
- link upperarm_Link: geometry collision mesh filename=package://grinding_descriptions/meshes/fr3v5/collision/uppe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; visual mesh filename=package://grinding_descriptions/meshes/fr3v5/visual/upperar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
- link wrist1_Link: geometry collision mesh filename=package://grinding_descriptions/meshes/fr3v5/collision/wris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; visual mesh filename=package://grinding_descriptions/meshes/fr3v5/visual/wrist1_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
- link wrist2_Link: geometry collision mesh filename=package://grinding_descriptions/meshes/fr3v5/collision/wris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; visual mesh filename=package://grinding_descriptions/meshes/fr3v5/visual/wrist2_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
- link wrist3_Link: geometry collision mesh filename=package://grinding_descriptions/meshes/fr3v5/collision/wris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; visual mesh filename=package://grinding_descriptions/meshes/fr3v5/visual/wrist3_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
