Commit message: Update

File: grinding_descriptions/urdf/cobotta/cobotta.urdf (robot description, URDF)
Before this commit: robot cobotta, 12 links, 11 joints
Links:
- removed link pestle
- removed link pestle_tip
- added link pedaee; visual mesh filename=package://grinding_descriptions/mesh/cobotta/jig_pedaee_140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
- added link pedaee_tip; visual box size=0 0 0
- link J1: mass 1 -> 1.29; geometry collision mesh filename=package://grinding_descriptions/urdf/cobotta/J1.dae scale=1 1 1; visual mesh filename=package://grinding_descriptions/urdf/cobotta/J1.dae scale=1 1 1
- link J2: mass 1 -> 0.39; geometry collision mesh filename=package://grinding_descriptions/urdf/cobotta/J2.dae scale=1 1 1; visual mesh filename=package://grinding_descriptions/urdf/cobotta/J2.dae scale=1 1 1
- link J3: mass 1 -> 0.35; geometry collision mesh filename=package://grinding_descriptions/urdf/cobotta/J3.dae scale=1 1 1; visual mesh filename=package://grinding_descriptions/urdf/cobotta/J3.dae scale=1 1 1
- link J4: mass 1 -> 0.35; geometry collision mesh filename=package://grinding_descriptions/urdf/cobotta/J4.dae scale=1 1 1; visual mesh filename=package://grinding_descriptions/urdf/cobotta/J4.dae scale=1 1 1
- link J5: mass 1 -> 0.19; geometry collision mesh filename=package://grinding_descriptions/urdf/cobotta/J5.dae scale=1 1 1; visual mesh filename=package://grinding_descriptions/urdf/cobotta/J5.dae scale=1 1 1
- link J6: mass 1 -> 0.03; geometry collision mesh filename=package://grinding_descriptions/urdf/cobotta/J6.dae scale=1 1 1; visual mesh filename=package://grinding_descriptions/urdf/cobotta/J6.dae scale=1 1 1
- link base_link: mass 1 -> 1.4; geometry collision mesh filename=package://grinding_descriptions/urdf/cobotta/base_link.dae scale=1 1 1; visual mesh filename=package://grinding_descriptions/urdf/cobotta/base_link.dae scale=1 1 1
Joints:
- removed joint joint_pestle
- removed joint joint_pestle_tip
- added joint joint_pedaee: type fixed, parent J6, child pedaee, origin xyz=0 0 0 rpy=0 0 0
- added joint joint_pedaee_tip: type fixed, parent pedaee, child pedaee_tip, origin xyz=0 0 0.160 rpy=0 0 0
- joint joint_1: limit lower=-2.617994 upper=2.617994 effort=1 velocity=1 -> lower=-2.617994 upper=2.617994 effort=1 velocity=0.383012504350156
- joint joint_2: limit lower=-1.047198 upper=1.745329 effort=1 velocity=1 -> lower=-1.047198 upper=1.745329 effort=1 velocity=0.37256670877697
- joint joint_3: limit lower=0.3141593 upper=2.443461 effort=1 velocity=1 -> lower=0.3141593 upper=2.443461 effort=1 velocity=0.68942250783028
- joint joint_4: limit lower=-2.96706 upper=2.96706 effort=1 velocity=1 -> lower=-2.96706 upper=2.96706 effort=1 velocity=0.702189591308619
- joint joint_5: limit lower=-1.658063 upper=2.356194 effort=1 velocity=1 -> lower=-1.658063 upper=2.356194 effort=1 velocity=0.702189591308619
- joint joint_6: limit lower=-2.96706 upper=2.96706 effort=1 velocity=1 -> lower=-2.96706 upper=2.96706 effort=1 velocity=1.05386470893922

File: grinding_descriptions/urdf/cobotta/setup_files/cobotta_description/cobotta.urdf (robot description, URDF)
Before this commit: robot cobotta, 12 links, 11 joints
Links:
- removed link pestle
- removed link pestle_tip
- added link pedaee; visual mesh filename=package://grinding_descriptions/mesh/cobotta/jig_pedaee_140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
- added link pedaee_tip; visual box size=0 0 0
- link J1: geometry collision mesh filename=package://grinding_descriptions/urdf/cobotta/J1.dae scale=1 1 1; visual mesh filename=package://grinding_descriptions/urdf/cobotta/J1.dae scale=1 1 1
- link J2: geometry collision mesh filename=package://grinding_descriptions/urdf/cobotta/J2.dae scale=1 1 1; visual mesh filename=package://grinding_descriptions/urdf/cobotta/J2.dae scale=1 1 1
- link J3: geometry collision mesh filename=package://grinding_descriptions/urdf/cobotta/J3.dae scale=1 1 1; visual mesh filename=package://grinding_descriptions/urdf/cobotta/J3.dae scale=1 1 1
- link J4: geometry collision mesh filename=package://grinding_descriptions/urdf/cobotta/J4.dae scale=1 1 1; visual mesh filename=package://grinding_descriptions/urdf/cobotta/J4.dae scale=1 1 1
- link J5: geometry collision mesh filename=package://grinding_descriptions/urdf/cobotta/J5.dae scale=1 1 1; visual mesh filename=package://grinding_descriptions/urdf/cobotta/J5.dae scale=1 1 1
- link J6: geometry collision mesh filename=package://grinding_descriptions/urdf/cobotta/J6.dae scale=1 1 1; visual mesh filename=package://grinding_descriptions/urdf/cobotta/J6.dae scale=1 1 1
- link base_link: geometry collision mesh filename=package://grinding_descriptions/urdf/cobotta/base_link.dae scale=1 1 1; visual mesh filename=package://grinding_descriptions/urdf/cobotta/base_link.dae scale=1 1 1
Joints:
- removed joint joint_pestle
- removed joint joint_pestle_tip
- added joint joint_pedaee: type fixed, parent J6, child pedaee, origin xyz=0 0 0 rpy=0 0 0
- added joint joint_pedaee_tip: type fixed, parent pedaee, child pedaee_tip, origin xyz=0 0 0.160 rpy=0 0 0

Commit message: Fix name

File: grinding_descriptions/urdf/cobotta/cobotta.urdf (robot description, URDF)
Before this commit: robot cobotta, 12 links, 11 joints
Links:
- removed link pedaee
- removed link pedaee_tip
- added link pestle; visual mesh filename=package://grinding_descriptions/mesh/cobotta/jig_pestle_140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
- added link pestle_tip; visual box size=0 0 0
Joints:
- removed joint joint_pedaee
- removed joint joint_pedaee_tip
- added joint joint_pestle: type fixed, parent J6, child pestle, origin xyz=0 0 0 rpy=0 0 0
- added joint joint_pestle_tip: type fixed, parent pestle, child pestle_tip, origin xyz=0 0 0.160 rpy=0 0 0

Commit message: Update urdf

File: grinding_descriptions/urdf/cobotta/cobotta.urdf (robot description, URDF)
Before this commit: robot cobotta, 12 links, 11 joints
Joints:
- joint joint_1: limit lower=-2.617994 upper=2.617994 effort=1 velocity=0.383012504350156 -> lower=-2.617994 upper=2.617994 effort=10 velocity=0.383012504350156; origin xyz=0.000000 0.000000 0.108000 rpy=0.000000 0.000000 0.000000 -> xyz=0.000000 0.000000 0.000000 rpy=0.000000 0.000000 0.000000
- joint joint_2: limit lower=-1.047198 upper=1.745329 effort=1 velocity=0.37256670877697 -> lower=-1.047198 upper=1.745329 effort=10 velocity=0.37256670877697
- joint joint_3: limit lower=0.3141593 upper=2.443461 effort=1 velocity=0.68942250783028 -> lower=0.3141593 upper=2.443461 effort=10 velocity=0.68942250783028
- joint joint_4: limit lower=-2.96706 upper=2.96706 effort=1 velocity=0.702189591308619 -> lower=-2.96706 upper=2.96706 effort=10 velocity=0.702189591308619
- joint joint_5: limit lower=-1.658063 upper=2.356194 effort=1 velocity=0.702189591308619 -> lower=-1.658063 upper=2.356194 effort=10 velocity=0.702189591308619
- joint joint_6: limit lower=-2.96706 upper=2.96706 effort=1 velocity=1.05386470893922 -> lower=-2.96706 upper=2.96706 effort=10 velocity=1.05386470893922

Commit message: Update urdf

File: grinding_descriptions/urdf/cobotta/cobotta.urdf (robot description, URDF)
Before this commit: robot cobotta, 12 links, 11 joints
Joints:
- joint joint_1: limit lower=-2.617994 upper=2.617994 effort=1 velocity=0.383012504350156 -> lower=-2.617994 upper=2.617994 effort=10 velocity=0.383012504350156; origin xyz=0.000000 0.000000 0.108000 rpy=0.000000 0.000000 0.000000 -> xyz=0.000000 0.000000  0.108000 rpy=0.000000 0.000000 0.000000
- joint joint_2: limit lower=-1.047198 upper=1.745329 effort=1 velocity=0.37256670877697 -> lower=-1.047198 upper=1.745329 effort=10 velocity=0.37256670877697
- joint joint_3: limit lower=0.3141593 upper=2.443461 effort=1 velocity=0.68942250783028 -> lower=0.3141593 upper=2.443461 effort=10 velocity=0.68942250783028
- joint joint_4: limit lower=-2.96706 upper=2.96706 effort=1 velocity=0.702189591308619 -> lower=-2.96706 upper=2.96706 effort=10 velocity=0.702189591308619
- joint joint_5: limit lower=-1.658063 upper=2.356194 effort=1 velocity=0.702189591308619 -> lower=-1.658063 upper=2.356194 effort=10 velocity=0.702189591308619
- joint joint_6: limit lower=-2.96706 upper=2.96706 effort=1 velocity=1.05386470893922 -> lower=-2.96706 upper=2.96706 effort=10 velocity=1.05386470893922

File: grinding_descriptions/urdf/cobotta/setup_files/cobotta.urdf.xacro (robot description, xacro)
@@ -71,6 +71,6 @@
 	<joint name="joint_1" type="revolute">
 		<parent link="base_link" />
-		<child link="J1" />
-		<origin rpy="0.000000 0.000000 0.000000" xyz="0.000000 0.000000 0.000000" />
+		<child link="J1" />grinding_descriptions/urdf/cobotta/setup_files/cobotta.urdf
+		<origin rpy="0.000000 0.000000 0.000000" xyz="0.000000 0.000000  0.108000" />
 		<axis xyz="-0.000000 -0.000000 1.000000" />
 		<limit effort="10" lower="-2.617994" upper="2.617994" velocity="0.383012504350156" />

Commit message: Update

File: grinding_descriptions/urdf/cobotta/cobotta.urdf (robot description, URDF)
Before this commit: robot cobotta, 12 links, 11 joints
Joints:
- joint joint_pestle_tip: origin xyz=0 0 0.160 rpy=0 0 0 -> xyz=0 0 0.159 rpy=0 0 0
- joint joint_spatula_tip: origin xyz=0.09 0 0 rpy=-1.57079632679 0 -1.57079632679 -> xyz=0.085 0 0 rpy=-1.57079632679 0 -1.57079632679
