Commit message: Add URDF for fr3v6 robot and update configurations
- Created a new URDF file for the fr3v6 robot, detailing its links, joints, and visual/collision geometries.
- Updated the planning scene configuration to reference the new move group name "fr3v6_arm".
- Modified the launch files to load the new fr3v6 URDF and associated MoveIt! configurations, ensuring compatibility with the updated robot model.

File: grinding_descriptions/urdf/fr3/fr3v6.urdf (robot description, URDF)
Before this commit: robot fr3v5, 13 links, 12 joints
Links:
- removed link forearm_Link
- removed link shoulder_Link
- removed link upperarm_Link
- removed link wrist1_Link
- removed link wrist2_Link
- removed link wrist3_Link
- added link j1_Link, mass 2.1225; collision mesh filename=package://frcobot_description/meshes/fr3v6/collision/j1_Lin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; visual mesh filename=package://frcobot_description/meshes/fr3v6/visual/j1_Link.D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
- added link j2_Link, mass 4.8053; collision mesh filename=package://frcobot_description/meshes/fr3v6/collision/j2_Lin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; visual mesh filename=package://frcobot_description/meshes/fr3v6/visual/j2_Link.D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
- added link j3_Link, mass 2.2312; collision mesh filename=package://frcobot_description/meshes/fr3v6/collision/j3_Lin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; visual mesh filename=package://frcobot_description/meshes/fr3v6/visual/j3_Link.D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
- added link j4_Link, mass 1.5961; collision mesh filename=package://frcobot_description/meshes/fr3v6/collision/j4_Lin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; visual mesh filename=package://frcobot_description/meshes/fr3v6/visual/j4_Link.D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
- added link j5_Link, mass 1.5961; collision mesh filename=package://frcobot_description/meshes/fr3v6/collision/j5_Lin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; visual mesh filename=package://frcobot_description/meshes/fr3v6/visual/j5_Link.D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
- added link j6_Link, mass 0.53877; collision mesh filename=package://frcobot_description/meshes/fr3v6/collision/j6_Lin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; visual mesh filename=package://frcobot_description/meshes/fr3v6/visual/j6_Link.D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
- link base_link: mass 0.77817 -> 0.78393; geometry collision mesh filename=package://frcobot_description/meshes/fr3v6/collision/base_l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; visual mesh filename=package://frcobot_description/meshes/fr3v6/visual/base_link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
Joints:
- joint j1: child shoulder_Link -> j1_Link
- joint j2: child upperarm_Link -> j2_Link; origin xyz=0 0 0.1392 rpy=1.5708 0 -1.4405E-05 -> xyz=0 0 0.14 rpy=1.5708 0 0; parent shoulder_Link -> j1_Link
- joint j3: child forearm_Link -> j3_Link; parent upperarm_Link -> j2_Link
- joint j4: child wrist1_Link -> j4_Link; parent forearm_Link -> j3_Link
- joint j5: child wrist2_Link -> j5_Link; origin xyz=0 0 0.10199 rpy=1.5708 1.4405E-05 0 -> xyz=0 0 0.102 rpy=1.5708 0 0; parent wrist1_Link -> j4_Link
- joint j6: child wrist3_Link -> j6_Link; parent wrist2_Link -> j5_Link
- joint tool: axis 0 0 0 -> 0 0 1; parent wrist3_Link -> j6_Link
